File: pcb/pcb-for-horse-collar/_restore_backup_2026-08-26T17-40-55-820/pcb-for-horse-collar.kicad_sch (KiCad schematic)
At the start: 29 parts, among them J1 Conn_01x02_Socket, P1 USB_C_Receptacle_USB2.0_16P, Q1 S8050, Q2 S8050, SW2 OS102011MS2Q, U1 ESP32-WROOM-32E, U2 BNO085, U3 CP2102N-Axx-xQFN28, U4 MCP73831-2-OT, U5 AP2112K-3.3

Commit message: First ok from gemini
Parts:
- removed R11, R12: 100 kΩ, Resistor_SMD:R_0805_2012Metric, symbol Device:R
- removed SW2: OS102011MS2Q, Button_Switch_THT:SW_Slide_SPDT_Straight_CK_OS102011MS2Q, symbol Switch:SW_SPDT
- added SW1: SW_SPST, Button_Switch_SMD:SW_DIP_SPSTx01_Slide_6.7x4.1mm_W6.73mm_P2.54mm_LowProfile_JPin, symbol Switch:SW_SPST
Connections:
- net VBAT+: now also SW1.2 (B)
- net VBAT_RAW: now also SW1.1 (A)
- no-connect marks 45 -> 46
Other:
- note removed: "System Components"
- moved on the sheet: U1
