File: pcb/pcb-for-horse-collar/pcb-for-horse-collar.kicad_sch (KiCad schematic)
At the start: 29 parts, among them J1 Conn_01x02_Socket, P1 USB_C_Receptacle_USB2.0_16P, Q1 S8050, Q2 S8050, SW2 OS102011MS2Q, U1 ESP32-WROOM-32E, U2 BNO085, U3 CP2102N-Axx-xQFN28, U4 MCP73831-2-OT, U5 AP2112K-3.3

Commit message: New size for edges
Parts:
- C1, C2, C3, C4, C5, C6, D1, R1, R10, R11, R12, R2, R3, R4, R5, R6, R7, R8, R9: KiLib_Generator (none) -> SMD_2terminal_chip_molded
- J1: KiLib_Generator (none) -> connector/JST
- Q1, Q2: footprint Package_TO_SOT_THT:TO-92_Inline -> Package_TO_SOT_SMD:SOT-23
- U3: KiLib_Generator (none) -> package/no_lead
- U4, U5: KiLib_Generator (none) -> package/gullwing
Connections:
- net unconnected-(P1-SHIELD-PadSH)_1: now reaches P1.SH (SHIELD)
